File: KiCad Files/MicroDev128.kicad_sch (KiCad schematic)
At the start: 27 parts, among them J1 UPDI Header, J3 GPIO, J4 PWR and ANALOG, SW1 SW_SP3T, SW2 RST, U1 AVR128DB32x-xRXB, U2 LT8653SEV_PBF, Y1 24MHz

Commit message: Updated for sponsor
Parts:
- removed C11, C12: 12pF, Capacitor_SMD:C_0402_1005Metric, symbol Device:C
- removed Y1: 24MHz, Crystal:Crystal_SMD_3225-4Pin_3.2x2.5mm, symbol Device:Crystal
Connections:
- net at U1.21 (XTAL32K2/PF1): now also R3.1
- net at J3.1 (Pin_1), U1.22 (PF2): no longer R3.1
Other:
- note removed: "Crystal Ocsilator"
